File: circuit/climobike.sch (KiCad schematic (older format))
At the start: 11 parts, among them IC1 ESP32-DevKitC, J1 Jack-DC, U1 DHT22, U2 Tiny_RTC_DS1307

Commit message: ADD: Full circuit schematic and pcb design
Parts:
- removed MQ3: MQ-X, symbol modules:MQ-X
- removed MQ5: MQ-Y, symbol modules:MQ-X
- added C1: 1000u, Capacitor_THT:CP_Radial_D10.0mm_P5.00mm, symbol Device:CP_Small
- added R1: R_SHUNT, Resistor_THT:R_Axial_DIN0207_L6.3mm_D2.5mm_P7.62mm_Horizontal, symbol Device:R
- added R2: LDR, OptoDevice:R_LDR_7x6mm_P5.1mm_Vertical, symbol Sensor_Optical:LDR03
- MQ1, MQ2, MQ4: footprint (none) -> Module:MQ-Sensor
Connections:
- net labels added: LDR_V
- net labels removed: CO_FLAG, MET_FLAG, TOX_FLAG, X_FLAG, X_OUT, Y_FLAG, Y_OUT
- no-connect marks 22 -> 31
Other:
- note added: "LIGHT SENSOR MODULE"
- note removed: "Extra MQ Gas Sensor Sockets\n"
- moved on the sheet: J1
